File: pcb/iCEboy-pcb.kicad_sch (KiCad schematic)
At the start: 64 parts, among them J1 DMG-CardEdge, J2 PROG_PORT, Q1 2N7002K, U1 TC74LCXR163245FT, U2 TC74LCXR163245FT, U3 ICE40UP5K-SG48ITR, U4 TPS79901DDCR, U5 TPS79901DDCR, U6 W25Q80DVSSIG, X1 SIT2001B 20MHz

Commit message: update schematic, change Lx to FBx, add LPF circuit for Vin, reselection of some components
Parts:
- removed L1, L2, L3: 600Ω, Inductor_SMD:L_0603_1608Metric, symbol Device:L
- removed R1: 10kΩ, Resistor_SMD:R_0603_1608Metric, symbol Device:R
- removed R9: DNP, Resistor_SMD:R_0603_1608Metric, symbol Device:R
- removed X1: SIT2001B 20MHz, Package_TO_SOT_SMD:SOT-23-5, symbol SIT2001B:SIT2001B
- added C17, C18: 1nF, Capacitor_SMD:C_0402_1005Metric, symbol Device:C
- added FB1, FB2, FB3: MPZ1608S601ATA00, Inductor_SMD:L_0603_1608Metric, symbol Device:FerriteBead
- added R8: 8.2kΩ, Resistor_SMD:R_0402_1005Metric, symbol Device:R
- added X1: SG-210STF 20MHz, Oscillator:Oscillator_SMD_SeikoEpson_SG210-4Pin_2.5x2.0mm, symbol Oscillator:SG-210STF
- C10, C12, C16, C2, C3, C4, C5, C6, C7, C8, C9: footprint Capacitor_SMD:C_0603_1608Metric -> Capacitor_SMD:C_0402_1005Metric
- C11: renamed from C15; footprint Capacitor_SMD:C_0603_1608Metric -> Capacitor_SMD:C_0402_1005Metric
- C13: renamed from C14; footprint Capacitor_SMD:C_0603_1608Metric -> Capacitor_SMD:C_0402_1005Metric
- C14: renamed from C13; footprint Capacitor_SMD:C_0603_1608Metric -> Capacitor_SMD:C_0402_1005Metric
- C15: renamed from C11; footprint Capacitor_SMD:C_0603_1608Metric -> Capacitor_SMD:C_0402_1005Metric
- C19: renamed from C17; value DNP -> 1uF; footprint Capacitor_SMD:C_0603_1608Metric -> Capacitor_SMD:C_0402_1005Metric
- C20: renamed from C18; footprint Capacitor_SMD:C_0603_1608Metric -> Capacitor_SMD:C_0402_1005Metric
- C21: renamed from C19; footprint Capacitor_SMD:C_0603_1608Metric -> Capacitor_SMD:C_0402_1005Metric
- C22: renamed from C20; footprint Capacitor_SMD:C_0603_1608Metric -> Capacitor_SMD:C_0402_1005Metric
- C23: renamed from C21; footprint Capacitor_SMD:C_0603_1608Metric -> Capacitor_SMD:C_0402_1005Metric
- C24: renamed from C22; footprint Capacitor_SMD:C_0603_1608Metric -> Capacitor_SMD:C_0402_1005Metric
- C25: renamed from C27; footprint Capacitor_SMD:C_0603_1608Metric -> Capacitor_SMD:C_0402_1005Metric
- C26: renamed from C24; footprint Capacitor_SMD:C_0603_1608Metric -> Capacitor_SMD:C_0402_1005Metric
- C27: renamed from C25; footprint Capacitor_SMD:C_0603_1608Metric -> Capacitor_SMD:C_0402_1005Metric
- C28: renamed from C23; footprint Capacitor_SMD:C_0603_1608Metric -> Capacitor_SMD:C_0402_1005Metric
- C30: renamed from C26; footprint Capacitor_SMD:C_0603_1608Metric -> Capacitor_SMD:C_0402_1005Metric
- R1: renamed from R2; footprint Resistor_SMD:R_0603_1608Metric -> Resistor_SMD:R_0402_1005Metric
- R10: renamed from R13; footprint Resistor_SMD:R_0603_1608Metric -> Resistor_SMD:R_0402_1005Metric
- R11, R12, R3: footprint Resistor_SMD:R_0603_1608Metric -> Resistor_SMD:R_0402_1005Metric
- R13: renamed from R14; footprint Resistor_SMD:R_0603_1608Metric -> Resistor_SMD:R_0402_1005Metric
- R14: renamed from R15; footprint Resistor_SMD:R_0603_1608Metric -> Resistor_SMD:R_0402_1005Metric
- R15: renamed from R16; footprint Resistor_SMD:R_0603_1608Metric -> Resistor_SMD:R_0402_1005Metric
- R2: renamed from R8; value DNP -> 8.2kΩ; footprint Resistor_SMD:R_0603_1608Metric -> Resistor_SMD:R_0402_1005Metric
- R4: renamed from R7; footprint Resistor_SMD:R_0603_1608Metric -> Resistor_SMD:R_0402_1005Metric
- R5: renamed from R4; footprint Resistor_SMD:R_0603_1608Metric -> Resistor_SMD:R_0402_1005Metric
- R6: renamed from R5; footprint Resistor_SMD:R_0603_1608Metric -> Resistor_SMD:R_0402_1005Metric
- R7: renamed from R6; footprint Resistor_SMD:R_0603_1608Metric -> Resistor_SMD:R_0402_1005Metric
- R9: renamed from R10; footprint Resistor_SMD:R_0603_1608Metric -> Resistor_SMD:R_0402_1005Metric
- renumbered C28 to C29, D2 to D1, D3 to D2, D4 to D3, D1 to D4
Connections:
- net +1V2: now also FB2.2
- net +3V3: now also FB3.2, X1.4 (Vcc)
- net +5V: now also FB1.2
- net 1V2VO: now also FB2.1
- net 3V3VO: now also FB3.1
- net CB-VIN: now also C19.1; no longer R2.1
- net DV-VIN: now also R2.2; no longer C19.2
- net GND: now also C17.2, C18.2, X1.2 (GND)
- net SYSCLK: now also X1.3 (OUT)
- net VCC: now also FB1.1
- new net: C17.1, R2.1, R8.2
- new net: C18.1, C19.2, R8.1
- no-connect marks 4 -> 5
Other:
- note added: "20kHz -40dB/dec LPF for audio input(Vin) WIP"
- moved on the sheet: C1, C10, C11, C12, C19, C21, C22, C24, C28, C30, Q1, R14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

Commit message: update pcb wip
Parts:
- removed D5: RSX101VAM-30TR, Diode_SMD:D_TUMD2, symbol Device:D
- added D5: BAT43XV2, Diode_SMD:D_SOD-523, symbol Device:D_Schottky
- U3: footprint Package_DFN_QFN:QFN-48-1EP_7x7mm_P0.5mm_EP5.6x5.6mm -> Package_DFN_QFN:QFN-48-1EP_7x7mm_P0.5mm_EP5.6x5.6mm_ThermalVias
Connections:
- net +3V3: now also D5.2 (A)
- net VPP: now also D5.1 (K)
Changed lines of the file:
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@@
       (effects (font (size 1.27 1.27)) (justify left))
     )
-    (property "Footprint" "Package_DFN_QFN:QFN-48-1EP_7x7mm_P0.5mm_EP5.6x5.6mm" (id 2) (at 204.47 105.41 0)
+    (property "Footprint" "Package_DFN_QFN:QFN-48-1EP_7x7mm_P0.5mm_EP5.6x5.6mm_ThermalVias" (id 2) (at 204.47 105.41 0)
       (effects (font (size 1.27 1.27)) hide)
     )
@@
     (property "Reference" "U3" (id 0) (at 200.66 129.54 0))
     (property "Value" "ICE40UP5K-SG48ITR" (id 1) (at 209.55 182.88 0))
-    (property "Footprint" "Package_DFN_QFN:QFN-48-1EP_7x7mm_P0.5mm_EP5.6x5.6mm" (id 2) (at 209.55 190.5 0)
+    (property "Footprint" "Package_DFN_QFN:QFN-48-1EP_7x7mm_P0.5mm_EP5.6x5.6mm_ThermalVias" (id 2) (at 209.55 190.5 0)
       (effects (font (size 1.27 1.27)) hide)
     )
@@
       (effects (font (size 1.27 1.27)) (justify left))
     )
-    (property "Footprint" "Package_DFN_QFN:QFN-48-1EP_7x7mm_P0.5mm_EP5.6x5.6mm" (id 2) (at 210.82 279.4 0)
+    (property "Footprint" "Package_DFN_QFN:QFN-48-1EP_7x7mm_P0.5mm_EP5.6x5.6mm_ThermalVias" (id 2) (at 210.82 279.4 0)
       (effects (font (size 1.27 1.27)) hide)
     )
@@
       (effects (font (size 1.27 1.27)) (justify left))
     )
-    (property "Footprint" "Package_DFN_QFN:QFN-48-1EP_7x7mm_P0.5mm_EP5.6x5.6mm" (id 2) (at 335.28 187.96 0)
+    (property "Footprint" "Package_DFN_QFN:QFN-48-1EP_7x7mm_P0.5mm_EP5.6x5.6mm_ThermalVias" (id 2) (at 335.28 187.96 0)
       (effects (font (size 1.27 1.27)) hide)
     )
@@
     (pin "1")
   )
-  (symbol (lib_id "Device:D") (at 323.85 140.97 180) (unit 1)
-    (in_bom yes) (on_board yes)
-    (property "Reference" "D5" (id 0) (at 323.85 135.4582 0))
-    (property "Value" "RSX101VAM-30TR" (id 1) (at 323.85 137.7696 0))
-    (property "Footprint" "Diode_SMD:D_TUMD2" (id 2) (at 323.85 140.97 0)
-      (effects (font (size 1.27 1.27)) hide)
-    )
-    (property "Datasheet" "~" (id 3) (at 323.85 140.97 0)
-      (effects (font (size 1.27 1.27)) hide)
-    )
-    (pin "1")
-    (pin "2")
-  )
   (symbol (lib_id "Device:C") (at 313.69 147.32 0) (unit 1)
     (in_bom yes) (on_board yes)
@@
     (pin "1")
   )
+  (symbol (lib_id "Device:D_Schottky") (at 323.85 140.97 0) (mirror y) (unit 1)
+    (in_bom yes) (on_board yes) (fields_autoplaced)
+    (property "Reference" "D5" (id 0) (at 324.1675 134.62 0))
+    (property "Value" "BAT43XV2" (id 1) (at 324.1675 137.16 0))
+    (property "Footprint" "Diode_SMD:D_SOD-523" (id 2) (at 323.85 140.97 0)
+      (effects (font (size 1.27 1.27)) hide)
+    )
+    (property "Datasheet" "~" (id 3) (at 323.85 140.97 0)
+      (effects (font (size 1.27 1.27)) hide)
+    )
+    (pin "1")
+    (pin "2")
+  )
   (symbol (lib_id "Device:C") (at 266.7 248.92 0) (unit 1)
     (in_bom yes) (on_board yes) (fields_autoplaced)
@@
       (reference "D4") (unit 1) (value "SML-E12Y8WT86") (footprint "LED_SMD:LED_0603_1608Metric_Castellated")
     )
-    (path "/00000000-0000-0000-0000-0000602b170a"
-      (reference "D5") (unit 1) (value "RSX101VAM-30TR") (footprint "Diode_SMD:D_TUMD2")
+    (path "/4f0cbadb-0dbf-4352-8aea-55a524e546d1"
+      (reference "D5") (unit 1) (value "BAT43XV2") (footprint "Diode_SMD:D_SOD-523")
     )
     (path "/218c812e-2ae6-44a2-aa8e-f477f8138079"
@@
     )
     (path "/00000000-0000-0000-0000-00005fbc12cf"
-      (reference "U3") (unit 1) (value "ICE40UP5K-SG48ITR") (footprint "Package_DFN_QFN:QFN-48-1EP_7x7mm_P0.5mm_EP5.6x5.6mm")
+      (reference "U3") (unit 1) (value "ICE40UP5K-SG48ITR") (footprint "Package_DFN_QFN:QFN-48-1EP_7x7mm_P0.5mm_EP5.6x5.6mm_ThermalVias")
     )
     (path "/00000000-0000-0000-0000-00005fbc1fb5"
-      (reference "U3") (unit 2) (value "ICE40UP5K-SG48ITR") (footprint "Package_DFN_QFN:QFN-48-1EP_7x7mm_P0.5mm_EP5.6x5.6mm")
+      (reference "U3") (unit 2) (value "ICE40UP5K-SG48ITR") (footprint "Package_DFN_QFN:QFN-48-1EP_7x7mm_P0.5mm_EP5.6x5.6mm_ThermalVias")
     )
     (path "/00000000-0000-0000-0000-00005fbc3d15"
-      (reference "U3") (unit 3) (value "ICE40UP5K-SG48ITR") (footprint "Package_DFN_QFN:QFN-48-1EP_7x7mm_P0.5mm_EP5.6x5.6mm")
+      (reference "U3") (unit 3) (value "ICE40UP5K-SG48ITR") (footprint "Package_DFN_QFN:QFN-48-1EP_7x7mm_P0.5mm_EP5.6x5.6mm_ThermalVias")
     )
     (path "/00000000-0000-0000-0000-00005fbc48f8"
-      (reference "U3") (unit 4) (value "ICE40UP5K-SG48ITR") (footprint "Package_DFN_QFN:QFN-48-1EP_7x7mm_P0.5mm_EP5.6x5.6mm")
+      (reference "U3") (unit 4) (value "ICE40UP5K-SG48ITR") (footprint "Package_DFN_QFN:QFN-48-1EP_7x7mm_P0.5mm_EP5.6x5.6mm_ThermalVias")
     )
     (path "/00000000-0000-0000-0000-00005fbf2ceb"

Commit message: change pin headers to THT, tweaking placement
Parts:
- U3: footprint Package_DFN_QFN:QFN-48-1EP_7x7mm_P0.5mm_EP5.6x5.6mm_ThermalVias -> Package_DFN_QFN:QFN-48-1EP_7x7mm_P0.5mm_EP5.6x5.6mm
Changed lines of the file:
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@@
       (effects (font (size 1.27 1.27)) (justify left))
     )
-    (property "Footprint" "Package_DFN_QFN:QFN-48-1EP_7x7mm_P0.5mm_EP5.6x5.6mm_ThermalVias" (id 2) (at 204.47 105.41 0)
+    (property "Footprint" "Package_DFN_QFN:QFN-48-1EP_7x7mm_P0.5mm_EP5.6x5.6mm" (id 2) (at 204.47 105.41 0)
       (effects (font (size 1.27 1.27)) hide)
     )
@@
     (property "Reference" "U3" (id 0) (at 200.66 129.54 0))
     (property "Value" "ICE40UP5K-SG48ITR" (id 1) (at 209.55 182.88 0))
-    (property "Footprint" "Package_DFN_QFN:QFN-48-1EP_7x7mm_P0.5mm_EP5.6x5.6mm_ThermalVias" (id 2) (at 209.55 190.5 0)
+    (property "Footprint" "Package_DFN_QFN:QFN-48-1EP_7x7mm_P0.5mm_EP5.6x5.6mm" (id 2) (at 209.55 190.5 0)
       (effects (font (size 1.27 1.27)) hide)
     )
@@
       (effects (font (size 1.27 1.27)) (justify left))
     )
-    (property "Footprint" "Package_DFN_QFN:QFN-48-1EP_7x7mm_P0.5mm_EP5.6x5.6mm_ThermalVias" (id 2) (at 210.82 279.4 0)
+    (property "Footprint" "Package_DFN_QFN:QFN-48-1EP_7x7mm_P0.5mm_EP5.6x5.6mm" (id 2) (at 210.82 279.4 0)
       (effects (font (size 1.27 1.27)) hide)
     )
@@
       (effects (font (size 1.27 1.27)) (justify left))
     )
-    (property "Footprint" "Package_DFN_QFN:QFN-48-1EP_7x7mm_P0.5mm_EP5.6x5.6mm_ThermalVias" (id 2) (at 335.28 187.96 0)
+    (property "Footprint" "Package_DFN_QFN:QFN-48-1EP_7x7mm_P0.5mm_EP5.6x5.6mm" (id 2) (at 335.28 187.96 0)
       (effects (font (size 1.27 1.27)) hide)
     )
@@
     )
     (path "/00000000-0000-0000-0000-00005fbc12cf"
-      (reference "U3") (unit 1) (value "ICE40UP5K-SG48ITR") (footprint "Package_DFN_QFN:QFN-48-1EP_7x7mm_P0.5mm_EP5.6x5.6mm_ThermalVias")
+      (reference "U3") (unit 1) (value "ICE40UP5K-SG48ITR") (footprint "Package_DFN_QFN:QFN-48-1EP_7x7mm_P0.5mm_EP5.6x5.6mm")
     )
     (path "/00000000-0000-0000-0000-00005fbc1fb5"
-      (reference "U3") (unit 2) (value "ICE40UP5K-SG48ITR") (footprint "Package_DFN_QFN:QFN-48-1EP_7x7mm_P0.5mm_EP5.6x5.6mm_ThermalVias")
+      (reference "U3") (unit 2) (value "ICE40UP5K-SG48ITR") (footprint "Package_DFN_QFN:QFN-48-1EP_7x7mm_P0.5mm_EP5.6x5.6mm")
     )
     (path "/00000000-0000-0000-0000-00005fbc3d15"
-      (reference "U3") (unit 3) (value "ICE40UP5K-SG48ITR") (footprint "Package_DFN_QFN:QFN-48-1EP_7x7mm_P0.5mm_EP5.6x5.6mm_ThermalVias")
+      (reference "U3") (unit 3) (value "ICE40UP5K-SG48ITR") (footprint "Package_DFN_QFN:QFN-48-1EP_7x7mm_P0.5mm_EP5.6x5.6mm")
     )
     (path "/00000000-0000-0000-0000-00005fbc48f8"
-      (reference "U3") (unit 4) (value "ICE40UP5K-SG48ITR") (footprint "Package_DFN_QFN:QFN-48-1EP_7x7mm_P0.5mm_EP5.6x5.6mm_ThermalVias")
+      (reference "U3") (unit 4) (value "ICE40UP5K-SG48ITR") (footprint "Package_DFN_QFN:QFN-48-1EP_7x7mm_P0.5mm_EP5.6x5.6mm")
     )
     (path "/00000000-0000-0000-0000-00005fbf2ceb"

Commit message: add mounting hole
Parts:
- added H1, H2, H3, H4: MH_2mm, MountingHole:MountingHole_2.1mm, symbol Mechanical:MountingHole
Changed lines of the file:
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@@
     (pin "2")
+  )
+  (symbol (lib_id "Mechanical:MountingHole") (at 434.34 22.86 0) (unit 1)
+    (in_bom yes) (on_board yes) (fields_autoplaced)
+    (property "Reference" "H1" (id 0) (at 436.88 21.5899 0)
+      (effects (font (size 1.27 1.27)) (justify left))
+    )
+    (property "Value" "MH_2mm" (id 1) (at 436.88 24.1299 0)
+      (effects (font (size 1.27 1.27)) (justify left))
+    )
+    (property "Footprint" "MountingHole:MountingHole_2.1mm" (id 2) (at 434.34 22.86 0)
+      (effects (font (size 1.27 1.27)) hide)
+    )
+    (property "Datasheet" "~" (id 3) (at 434.34 22.86 0)
+      (effects (font (size 1.27 1.27)) hide)
+    )
   )
   (symbol (lib_id "power:+1V2") (at 459.74 6.35 0) (unit 1)
@@
     (pin "1")
   )
+  (symbol (lib_id "Mechanical:MountingHole") (at 434.34 33.02 0) (unit 1)
+    (in_bom yes) (on_board yes) (fields_autoplaced)
+    (property "Reference" "H3" (id 0) (at 436.88 31.7499 0)
+      (effects (font (size 1.27 1.27)) (justify left))
+    )
+    (property "Value" "MH_2mm" (id 1) (at 436.88 34.2899 0)
+      (effects (font (size 1.27 1.27)) (justify left))
+    )
+    (property "Footprint" "MountingHole:MountingHole_2.1mm" (id 2) (at 434.34 33.02 0)
+      (effects (font (size 1.27 1.27)) hide)
+    )
+    (property "Datasheet" "~" (id 3) (at 434.34 33.02 0)
+      (effects (font (size 1.27 1.27)) hide)
+    )
+  )
+  (symbol (lib_id "Mechanical:MountingHole") (at 434.34 27.94 0) (unit 1)
+    (in_bom yes) (on_board yes) (fields_autoplaced)
+    (property "Reference" "H2" (id 0) (at 436.88 26.6699 0)
+      (effects (font (size 1.27 1.27)) (justify left))
+    )
+    (property "Value" "MH_2mm" (id 1) (at 436.88 29.2099 0)
+      (effects (font (size 1.27 1.27)) (justify left))
+    )
+    (property "Footprint" "MountingHole:MountingHole_2.1mm" (id 2) (at 434.34 27.94 0)
+      (effects (font (size 1.27 1.27)) hide)
+    )
+    (property "Datasheet" "~" (id 3) (at 434.34 27.94 0)
+      (effects (font (size 1.27 1.27)) hide)
+    )
+  )
   (symbol (lib_id "Device:R") (at 260.35 242.57 270) (unit 1)
     (in_bom yes) (on_board yes)
@@
     (pin "1")
   )
+  (symbol (lib_id "Mechanical:MountingHole") (at 434.34 38.1 0) (unit 1)
+    (in_bom yes) (on_board yes) (fields_autoplaced)
+    (property "Reference" "H4" (id 0) (at 436.88 36.8299 0)
+      (effects (font (size 1.27 1.27)) (justify left))
+    )
+    (property "Value" "MH_2mm" (id 1) (at 436.88 39.3699 0)
+      (effects (font (size 1.27 1.27)) (justify left))
+    )
+    (property "Footprint" "MountingHole:MountingHole_2.1mm" (id 2) (at 434.34 38.1 0)
+      (effects (font (size 1.27 1.27)) hide)
+    )
+    (property "Datasheet" "~" (id 3) (at 434.34 38.1 0)
+      (effects (font (size 1.27 1.27)) hide)
+    )
+  )
   (symbol (lib_id "power:PWR_FLAG") (at 447.04 6.35 180) (unit 1)
     (in_bom yes) (on_board yes) (fields_autoplaced)
@@
       (reference "FB3") (unit 1) (value "MPZ1608S601ATA00") (footprint "Inductor_SMD:L_0603_1608Metric")
     )
+    (path "/2f4d4976-44f2-4b4d-832b-e65621c2ec1b"
+      (reference "H1") (unit 1) (value "MH_2mm") (footprint "MountingHole:MountingHole_2.1mm")
+    )
+    (path "/9f51ca48-589e-4a68-b113-010385c405ef"
+      (reference "H2") (unit 1) (value "MH_2mm") (footprint "MountingHole:MountingHole_2.1mm")
+    )
+    (path "/9b1529b3-c025-495c-8a91-dd8b2dfefaae"
+      (reference "H3") (unit 1) (value "MH_2mm") (footprint "MountingHole:MountingHole_2.1mm")
+    )
+    (path "/cd37b72a-e81d-49c9-a313-fb067d22b828"
+      (reference "H4") (unit 1) (value "MH_2mm") (footprint "MountingHole:MountingHole_2.1mm")
+    )
     (path "/00000000-0000-0000-0000-00005fc7ddc7"

Commit message: add reverse current protection circuit between VCC and 5V, remove mounthole
Parts:
- removed FB1: MPZ1608S601ATA00, Inductor_SMD:L_0603_1608Metric, symbol Device:FerriteBead
- removed H1, H2, H3, H4: MH_2mm, MountingHole:MountingHole_2.1mm, symbol Mechanical:MountingHole
- added Q1: DMG3415U, Package_TO_SOT_SMD:SOT-23, symbol Device:Q_PMOS_GSD
- added Q2: HN4A56JU, Package_TO_SOT_SMD:SOT-353_SC-70-5, symbol HN4A56JU:HN4A56JU
- added R1, R3: 12kΩ, Resistor_SMD:R_0402_1005Metric, symbol Device:R
- added R2: DNP, Resistor_SMD:R_0603_1608Metric, symbol Device:R
- renumbered C21 to C20, C22 to C21, C20 to C22, C24 to C23, C23 to C24, C28 to C26, C26 to C27, C27 to C28, C30 to C29, C29 to C30, FB2 to FB1, FB3 to FB2, Q1 to Q3, R7 to R10, R8 to R11, R9 to R12, R10 to R13, R11 to R14, R12 to R15, R14 to R16, R15 to R17, R13 to R18, R1 to R4, R2 to R5, R3 to R6, R4 to R7, R5 to R8, R6 to R9
Connections:
- net +5V: now also Q1.2 (S), Q2.3 (E2), R2.2
- net GND: now also R1.2, R3.2
- net VCC: now also Q1.3 (D), Q2.1 (E1), R2.1
- new net: Q2.2 (B), Q2.5 (C1), R1.1
- new net: Q1.1 (G), Q2.4 (C2), R3.1
Other:
- note added: "20kHz -40dB/dec LPF for audio input(VIN)"
- note removed: "20kHz -40dB/dec LPF for audio input(Vin) WIP"
- moved on the sheet: C1
