File: pcb/midi/tGB-midi.kicad_pcb (KiCad board)
At the start: 2 copper layers, 25.2 x 31 mm, 25 parts, among them J1 MIDI_IN, J2 MIDI_THRU, J3 MIDI_OUT, J4 IO, U1 TLP2368, U2 TC7WZ07FK

Commit message: update pcb (wip)
Parts:
- moved C3 12.7 mm to (77.0, 89.9)
- moved FB2 12.7 mm to (64.2, 83.8)
- moved FB3 12.7 mm to (76.9, 83.8)
- moved R2 12.7 mm to (76.9, 86.3)
- moved R6 12.7 mm to (75.9, 89.9)
- moved U1 12.7 mm to (70.2, 90.2)
- moved U2 12.7 mm to (79.2, 90.2)
- moved C1 12.7 mm to (61.9, 83.3)
- moved J4 12.7 mm to (61.2, 98.0)
- moved C4 12.7 mm to (63.5, 93.4)
- moved D1 12.7 mm to (64.9, 89.6)
- moved FB1 12.7 mm to (66.3, 83.8)
- moved FB4 12.7 mm to (74.8, 83.8)
- moved FB5 12.7 mm to (81.1, 83.8)
- moved FB6 12.7 mm to (83.3, 83.8)
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
Commit message: fix silkscreens
Other:
- board text added: "3.3V"
- board text added: "5V"
- board text removed: "+3.3V"
- board text removed: "+5V"
Changed lines of the file:
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@@
     (effects (font (size 0.6 0.6) (thickness 0.12)) (justify mirror))
   )
-  (gr_text "+5V" (at 61.17 97.3) (layer "B.SilkS")
+  (gr_text "5V" (at 61.17 97.3) (layer "B.SilkS")
     (effects (font (size 0.6 0.6) (thickness 0.12)) (justify mirror))
   )
@@
     (effects (font (size 0.6 0.6) (thickness 0.12)) (justify mirror))
   )
-  (gr_text "+3.3V" (at 63.71 97.3) (layer "B.SilkS")
+  (gr_text "3.3V" (at 63.71 97.3) (layer "B.SilkS")
     (effects (font (size 0.6 0.6) (thickness 0.12)) (justify mirror))
   )
@@
     (effects (font (size 0.6 0.6) (thickness 0.12)))
   )
-  (gr_text "+3.3V" (at 63.71 95.8) (layer "F.SilkS")
+  (gr_text "3.3V" (at 63.71 95.8) (layer "F.SilkS")
     (effects (font (size 0.6 0.6) (thickness 0.12)))
   )
@@
     (effects (font (size 0.6 0.6) (thickness 0.12)))
   )
-  (gr_text "+5V" (at 61.17 95.8) (layer "F.SilkS")
+  (gr_text "5V" (at 61.17 95.8) (layer "F.SilkS")
     (effects (font (size 0.6 0.6) (thickness 0.12)))
   )

Commit message: add silkscreen of board name
Other:
- board text added: "Rev.A 2022-09"
- board text added: "tGB MIDI Adapter"
Changed lines of the file:
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@@
   (gr_line (start 78.75 95.735) (end 78.95 95.535) (layer "F.SilkS") (width 0.12))
   (gr_line (start 78.95 95.535) (end 78.95 96.025) (layer "F.SilkS") (width 0.12))
+  (gr_arc (start 85 69) (mid 85.141421 69.058579) (end 85.2 69.2) (layer "Edge.Cuts") (width 0.1))
   (gr_line (start 60 69.2) (end 60 99.8) (layer "Edge.Cuts") (width 0.1))
   (gr_line (start 60.2 100) (end 85 100) (layer "Edge.Cuts") (width 0.1))
@@
   (gr_arc (start 60.2 100) (mid 60.058579 99.941421) (end 60 99.8) (layer "Edge.Cuts") (width 0.1))
   (gr_arc (start 85.2 99.8) (mid 85.141421 99.941421) (end 85 100) (layer "Edge.Cuts") (width 0.1))
-  (gr_arc (start 85 69) (mid 85.141421 69.058579) (end 85.2 69.2) (layer "Edge.Cuts") (width 0.1))
   (gr_line (start 85 69) (end 60.2 69) (layer "Edge.Cuts") (width 0.1))
   (gr_text "GND" (at 66.25 97.3) (layer "B.SilkS")
@@
     (effects (font (size 0.6 0.6) (thickness 0.12)) (justify mirror))
   )
+  (gr_text "tGB MIDI Adapter" (at 84.2 90 270) (layer "B.SilkS")
+    (effects (font (size 0.6 0.6) (thickness 0.12)) (justify mirror))
+  )
   (gr_text "MIDI" (at 72.6 71.5) (layer "B.SilkS")
     (effects (font (size 0.6 0.6) (thickness 0.12)) (justify mirror))
   )
   (gr_text "IN" (at 64.15 70.2) (layer "B.SilkS")
+    (effects (font (size 0.6 0.6) (thickness 0.12)) (justify mirror))
+  )
+  (gr_text "Rev.A  2022-09" (at 61 90 270) (layer "B.SilkS")
     (effects (font (size 0.6 0.6) (thickness 0.12)) (justify mirror))
   )
@@
   (via (at 64.39 92.94) (size 0.8) (drill 0.4) (layers "F.Cu" "B.Cu") (net 1))
   (segment (start 61.9 82.82) (end 61.9 80) (width 0.25) (layer "F.Cu") (net 2))
-  (segment (start 75.9 90.385) (end 75.9 91.63) (width 0.5) (layer "F.Cu") (net 3))
   (segment (start 75.9 90.385) (end 76.95 90.385) (width 0.5) (layer "F.Cu") (net 3))
+  (segment (start 75.9 91.63) (end 73.63 93.9) (width 0.5) (layer "F.Cu") (net 3))
   (segment (start 70.76 92.95) (end 70.76 93.9) (width 0.5) (layer "F.Cu") (net 3))
+  (segment (start 73.63 93.9) (end 62.95 93.9) (width 0.5) (layer "F.Cu") (net 3))
+  (segment (start 61.65 95.2) (end 61.65 97.57) (width 0.5) (layer "F.Cu") (net 3))
   (segment (start 74.52 88.88) (end 74.8 88.6) (width 0.5) (layer "F.Cu") (net 3))
   (segment (start 70.76 92.95) (end 70.76 90) (width 0.5) (layer "F.Cu") (net 3))
-  (segment (start 75.9 91.63) (end 73.63 93.9) (width 0.5) (layer "F.Cu") (net 3))
   (segment (start 74.8 88.6) (end 74.8 86.86) (width 0.5) (layer "F.Cu") (net 3))
   (segment (start 71.88 88.88) (end 73.3 88.88) (width 0.5) (layer "F.Cu") (net 3))
   (segment (start 76.95 90.385) (end 80.315 90.385) (width 0.5) (layer "F.Cu") (net 3))
-  (segment (start 73.63 93.9) (end 62.95 93.9) (width 0.5) (layer "F.Cu") (net 3))
-  (segment (start 61.17 95.68) (end 61.17 98.05) (width 0.5) (layer "F.Cu") (net 3))
+  (segment (start 75.9 90.385) (end 75.9 91.63) (width 0.5) (layer "F.Cu") (net 3))
+  (segment (start 62.95 93.9) (end 61.65 95.2) (width 0.5) (layer "F.Cu") (net 3))
+  (segment (start 61.65 97.57) (end 61.17 98.05) (width 0.5) (layer "F.Cu") (net 3))
   (segment (start 70.76 90) (end 71.88 88.88) (width 0.5) (layer "F.Cu") (net 3))
   (segment (start 83.3 87.4) (end 83.3 86.86) (width 0.5) (layer "F.Cu") (net 3))
   (segment (start 79.9 91.7) (end 79.9 90.385) (width 0.25) (layer "F.Cu") (net 3))
   (segment (start 80.315 90.385) (end 83.3 87.4) (width 0.5) (layer "F.Cu") (net 3))
-  (segment (start 62.95 93.9) (end 61.17 95.68) (width 0.5) (layer "F.Cu") (net 3))
   (segment (start 73.3 88.88) (end 74.52 88.88) (width 0.5) (layer "F.Cu") (net 3))
   (segment (start 64.925 87.675) (end 64.925 88.88) (width 0.25) (layer "F.Cu") (net 4))
@@
   (segment (start 83.3 85.84) (end 83.3 84.5875) (width 0.25) (layer "F.Cu") (net 16))
   (segment (start 77.88 93.65) (end 76.85 93.65) (width 0.5) (layer "F.Cu") (net 17))
-  (segment (start 63.71 95.69) (end 63.71 98.05) (width 0.5) (layer "F.Cu") (net 17))
-  (segment (start 73.95 94.8) (end 64.6 94.8) (width 0.5) (layer "F.Cu") (net 17))
-  (segment (start 64.6 94.8) (end 63.71 95.69) (width 0.5) (layer "F.Cu") (net 17))
   (segment (start 75.1 93.65) (end 73.95 94.8) (width 0.5) (layer "F.Cu") (net 17))
+  (segment (start 65.2 94.8) (end 64.2 95.8) (width 0.5) (layer "F.Cu") (net 17))
+  (segment (start 73.95 94.8) (end 65.2 94.8) (width 0.5) (layer "F.Cu") (net 17))
   (segment (start 76.85 93.65) (end 75.1 93.65) (width 0.5) (layer "F.Cu") (net 17))
+  (segment (start 64.2 97.56) (end 63.71 98.05) (width 0.5) (layer "F.Cu") (net 17))
+  (segment (start 64.2 95.8) (end 64.2 97.56) (width 0.5) (layer "F.Cu") (net 17))
   (segment (start 79.235 90.96) (end 77.94 90.96) (width 0.25) (layer "F.Cu") (net 18))
   (segment (start 79.4 91.7) (end 79.4 91.125) (width 0.25) (layer "F.Cu") (net 18))
-  (segment (start 79.4 91.7) (end 79.4 92.785) (width 0.25) (layer "F.Cu") (net 18))
-  (segment (start 81.49 94.875) (end 81.49 98.05) (width 0.25) (layer "F.Cu") (net 18))
+  (segment (start 80.9 97.46) (end 81.49 98.05) (width 0.25) (layer "F.Cu") (net 18))
+  (segment (start 79.4 92.785) (end 80.9 94.285) (width 0.25) (layer "F.Cu") (net 18))
+  (segment (start 80.9 94.285) (end 80.9 97.46) (width 0.25) (layer "F.Cu") (net 18))
   (segment (start 77.94 90.96) (end 76.85 92.05) (width 0.25) (layer "F.Cu") (net 18))
   (segment (start 79.4 91.125) (end 79.235 90.96) (width 0.25) (layer "F.Cu") (net 18))
-  (segment (start 79.4 92.785) (end 81.49 94.875) (width 0.25) (layer "F.Cu") (net 18))
+  (segment (start 79.4 91.7) (end 79.4 92.785) (width 0.25) (layer "F.Cu") (net 18))
   (segment (start 76.85 92.05) (end 76.85 92.63) (width 0.25) (layer "F.Cu") (net 18))
   (segment (start 78.9 93.65) (end 78.9 91.7) (width 0.25) (layer "F.Cu") (net 19))
